File: Hardware/RedBoard_Turbo.brd (EAGLE design)
At the start: 58.4 x 53.3 mm, 149 parts, among them Q1 2.5A/30V, Q2 2N7002PW, U1 MCP73831, U2 74AHC1G125, U3 3.3V, U4 ATSAMD21G-A, U5 W25Q32FV, Y1 32.768kHz

Commit message: Updated schematic
Updated part names and removed extra text
Parts:
- renumbered S2 to S1, SJ2 to SJ1
Changed lines of the file:
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@@
 <layer number="49" name="Reference" color="7" fill="1" visible="no" active="yes"/>
 <layer number="50" name="dxf" color="7" fill="1" visible="no" active="yes"/>
-<layer number="51" name="tDocu" color="6" fill="1" visible="no" active="yes"/>
+<layer number="51" name="tDocu" color="6" fill="1" visible="yes" active="yes"/>
 <layer number="52" name="bDocu" color="6" fill="1" visible="no" active="yes"/>
 <layer number="91" name="Nets" color="2" fill="1" visible="no" active="no"/>
@@
 <attribute name="VALUE" x="2.794" y="24.892" size="0.4064" layer="27" font="vector"/>
 </element>
-<element name="SJ2" library="SparkFun-Passives" package="PAD-JUMPER-2-NC_BY_TRACE_NO_SILK" value="PWR-LED" x="6.35" y="34.925" smashed="yes" rot="MR180">
+<element name="SJ1" library="SparkFun-Passives" package="PAD-JUMPER-2-NC_BY_TRACE_NO_SILK" value="PWR-LED" x="6.35" y="34.925" smashed="yes" rot="MR180">
 <attribute name="NAME" x="6.35" y="34.036" size="0.4064" layer="26" rot="MR180" align="bottom-center"/>
 <attribute name="VALUE" x="6.35" y="35.814" size="0.4064" layer="28" rot="MR180" align="top-center"/>
@@
 <element name="U$85" library="buzzard_labels" package="REDBOARD_TURBO1" value="" x="34.036" y="45.466" rot="MR270"/>
 <element name="U$87" library="buzzard_labels (1)" package="CHG_SET1" value="" x="24.511" y="21.59" rot="MR270"/>
-<element name="S2" library="SparkFun-Switches" package="TACTILE_SWITCH_SMD_5.2MM" value="" x="47.879" y="10.795">
+<element name="S1" library="SparkFun-Switches" package="TACTILE_SWITCH_SMD_5.2MM" value="" x="47.879" y="10.795">
 <attribute name="PROD_ID" value="SWCH-14139" x="47.879" y="10.795" size="1.778" layer="27" display="off"/>
 </element>
@@
 <contactref element="JP6" pad="5"/>
 <contactref element="U2" pad="3"/>
-<contactref element="SJ2" pad="1"/>
+<contactref element="SJ1" pad="1"/>
 <contactref element="JP7" pad="GND@1"/>
 <contactref element="JP3" pad="GND"/>
@@
 <wire x1="44.831" y1="28.956" x2="44.87" y2="28.995" width="0.254" layer="1"/>
 <wire x1="44.87" y1="28.995" x2="45.847" y2="28.995" width="0.254" layer="1"/>
-<contactref element="S2" pad="3"/>
-<contactref element="S2" pad="4"/>
+<contactref element="S1" pad="3"/>
+<contactref element="S1" pad="4"/>
 </signal>
 <signal name="3.3V">
@@
 <wire x1="50.673" y1="13.97" x2="49.53" y2="13.97" width="0.2032" layer="1"/>
 <wire x1="38.989" y1="12.1285" x2="38.989" y2="3.429" width="0.2032" layer="16"/>
-<contactref element="S2" pad="1"/>
-<contactref element="S2" pad="2"/>
+<contactref element="S1" pad="1"/>
+<contactref element="S1" pad="2"/>
 <wire x1="38.989" y1="12.1285" x2="37.4015" y2="12.1285" width="0.2032" layer="16"/>
 <wire x1="50.673" y1="12.7" x2="50.673" y2="13.97" width="0.2032" layer="1"/>
@@
 <signal name="N$12">
 <contactref element="D3" pad="C"/>
-<contactref element="SJ2" pad="2"/>
+<contactref element="SJ1" pad="2"/>
 <wire x1="4.687" y1="34.925" x2="4.687" y2="35.929" width="0.2032" layer="1"/>
 <wire x1="4.687" y1="35.929" x2="4.826" y2="36.068" width="0.2032" layer="1"/>
