File: Hardware/Production/RedBoard_Turbo-Panel.brd (EAGLE design)
At the start: 58.4 x 53.3 mm, 149 parts, among them Q1 2.5A/30V, Q2 2N7002PW, U1 MCP73831, U2 74AHC1G125, U3 3.3V, U4 ATSAMD21G-A, U5 W25Q32FV, Y1 32.768kHz

Commit message: panel
Parts:
- removed FRAME1: FRAME-LEDGER, SparkFun-Aesthetics:CREATIVE_COMMONS
- added C100, C101, C102, C107, C111, C112, C113, C114, C115, C116, C121, C125, C126, C15, C16, C17, C18, C23, C27, C28, C29, C30, C31, C32, C37, C41, C42, C43, C44, C45, C46, C51, C55, C56, C57, C58, C59, C60, C65, C69, C70, C71, C72, C73, C74, C79, C83, C84, C85, C86, C87, C88, C93, C97, C98, C99: 0.1uF, SparkFun-Capacitors:0603-CAP
- added C103, C104, C117, C118, C19, C20, C33, C34, C47, C48, C61, C62, C75, C76, C89, C90: 15pF, SparkFun-Capacitors:0603-CAP
- added C105, C119, C21, C35, C49, C63, C77, C91: 1.0uF, SparkFun-Capacitors:0805
- added C106, C120, C22, C36, C50, C64, C78, C92: 2.2uF, SparkFun-Capacitors:0603-CAP
- added C108, C122, C24, C38, C52, C66, C80, C94: 2.2UF, SparkFun-Capacitors:1206@1
- added C109, C110, C123, C124, C25, C26, C39, C40, C53, C54, C67, C68, C81, C82, C95, C96: 4.7uF, SparkFun-Capacitors:0603-CAP
- added D10, D17, D24, D31, D38, D45, D52, D59: BLUE, SparkFun-LED:LED-0603
- added D11, D12, D18, D19, D25, D26, D32, D33, D39, D40, D46, D47, D53, D54, D60, D61: Yellow, SparkFun-LED:LED-0603
- added D13, D20, D27, D34, D41, D48, D55, D62: BAT20J, SparkFun-DiscreteSemi:SOD-323
- added D14, D21, D28, D35, D42, D49, D56, D63: WS2812B, SparkFun-LED:WS2812B
- added D15, D22, D29, D36, D43, D50, D57, D8: GREEN, SparkFun-LED:LED-0603
- added D16, D23, D30, D37, D44, D51, D58, D9: RED, SparkFun-LED:LED-0603
- added E$1, E$2: (no value), SparkFun-Aesthetics:FIDUCIAL-1X2
- added E$3: (no value), SparkFun-Retired:FIDUCIAL-1.5X3
- added F2, F3, F4, F5, F6, F7, F8, F9: 500mA, SparkFun-PowerIC:PTC-1206
- added FID10, FID11, FID12, FID13, FID14, FID15, FID16, FID17, FID18, FID19, FID20, FID21, FID22, FID23, FID24, FID25, FID26, FID27, FID28, FID29, FID30, FID31, FID32, FID33, FID34, FID35, FID36, FID5, FID6, FID7, FID8, FID9: FIDUCIAL1X2, SparkFun-Aesthetics:FIDUCIAL-1X2
- added J10, J13, J16, J19, J22, J25, J4, J7: (no value), SparkFun-Connectors:JST-2-PTH
- added J11, J14, J17, J20, J23, J26, J5, J8: (no value), SparkFun-Connectors:1X04_1MM_RA
- added J12, J15, J18, J21, J24, J27, J6, J9: (no value), SparkFun-Connectors:USB-MICROB-PTH-MILL
- added JP1, JP10, JP13, JP16, JP19, JP22, JP25, JP5: CORTEX_DEBUGPTH, samd21-temp:2X5-PTH-1.27MM
- added JP11, JP14, JP17, JP2, JP20, JP23, JP26, JP8: ARDUINO_UNO_R3LOCK_HOLES, SparkFun-Boards:ARDUINO_R3_LOCK_HOLES
- added JP12, JP15, JP18, JP21, JP24, JP27, JP4, JP9: POWER_JACKPTH, SparkFun-Connectors:POWER_JACK_PTH
- added L2, L3, L4, L5, L6, L7, L8, L9: FB - 30Ohm, SparkFun-Passives:0603
- added LOGO10, LOGO14, LOGO18, LOGO22, LOGO26, LOGO30, LOGO34, LOGO6: SFE_LOGO_NAME_FLAME.2_INCH, SparkFun-Aesthetics:SFE_LOGO_NAME_FLAME_.2
- added LOGO11, LOGO15, LOGO19, LOGO23, LOGO27, LOGO31, LOGO35, LOGO7: SFE_LOGO_NAME_FLAME.3_INCH, SparkFun-Aesthetics:SFE_LOGO_NAME_FLAME_.3
- added LOGO12, LOGO16, LOGO20, LOGO24, LOGO28, LOGO32, LOGO36, LOGO8: OSHW-LOGOL, SparkFun-Aesthetics:OSHW-LOGO-L
- added LOGO13, LOGO17, LOGO21, LOGO25, LOGO29, LOGO33, LOGO5, LOGO9: OSHW-LOGOS, SparkFun-Aesthetics:OSHW-LOGO-S
- added Q10, Q12, Q14, Q16, Q18, Q4, Q6, Q8: 2.5A/30V, SparkFun-DiscreteSemi:SOT23-3
- added Q11, Q13, Q15, Q17, Q3, Q5, Q7, Q9: 2N7002PW, SparkFun-DiscreteSemi:SOT323
- added R100, R108, R16, R24, R28, R36, R40, R48, R52, R60, R64, R72, R76, R84, R88, R96: 100k, SparkFun-Resistors:0603-RES
- added R101, R102, R104, R106, R14, R15, R17, R18, R20, R22, R26, R27, R29, R30, R32, R34, R38, R39, R41, R42, R44, R46, R50, R51, R53, R54, R56, R58, R62, R63, R65, R66, R68, R70, R74, R75, R77, R78, R80, R82, R86, R87, R89, R90, R92, R94, R98, R99: 330, SparkFun-Resistors:0603-RES
- added R103, R19, R31, R43, R55, R67, R79, R91: 47K, SparkFun-Resistors:0603-RES
- added R105, R21, R33, R45, R57, R69, R81, R93: 3.9K, SparkFun-Resistors:0603
- added R107, R23, R35, R47, R59, R71, R83, R95: PROG, SparkFun-Passives:1/6W-RES
- added R13, R25, R37, R49, R61, R73, R85, R97: 10K, SparkFun-Resistors:0603-RES
- added S2, S3, S4, S5, S6, S7, S8, S9: (no value), SparkFun-Switches:TACTILE_SWITCH_SMD_5.2MM
- added SJ2, SJ3, SJ4, SJ5, SJ6, SJ7, SJ8, SJ9: PWR-LED, SparkFun-Passives:PAD-JUMPER-2-NC_BY_TRACE_NO_SILK
- added TP2, TP3, TP4, TP5, TP6, TP7, TP8, TP9: TEST-POINTTP_15TH_THRU, SparkFun-Connectors:TP_15TH
- added U$100, U$188, U$276, U$364, U$452, U$540, U$628, U$716: (no value), buzzard_labels (22):D87
- added U$101, U$189, U$277, U$365, U$453, U$541, U$629, U$717: (no value), buzzard_labels (22):D96
- added U$102, U$190, U$278, U$366, U$454, U$542, U$630, U$718: (no value), buzzard_labels (22):D105
- added U$103, U$191, U$279, U$367, U$455, U$543, U$631, U$719: (no value), buzzard_labels (22):D114
- added U$104, U$192, U$280, U$368, U$456, U$544, U$632, U$720: (no value), buzzard_labels (22):D123
- added U$105, U$193, U$281, U$369, U$457, U$545, U$633, U$721: (no value), buzzard_labels (22):D132
- added U$106, U$121, U$122, U$194, U$209, U$210, U$282, U$297, U$298, U$370, U$385, U$386, U$458, U$473, U$474, U$546, U$561, U$562, U$634, U$649, U$650, U$722, U$737, U$738: (no value), buzzard_labels (22):GND16
- added U$107, U$195, U$283, U$371, U$459, U$547, U$635, U$723: (no value), buzzard_labels (22):SDA1
- added U$108, U$196, U$284, U$372, U$460, U$548, U$636, U$724: (no value), buzzard_labels (22):SCL0
- added U$109, U$197, U$285, U$373, U$461, U$549, U$637, U$725: (no value), buzzard_labels (22):TX28
- added U$110, U$198, U$286, U$374, U$462, U$550, U$638, U$726: (no value), buzzard_labels (22):RX29
- added U$111, U$199, U$287, U$375, U$463, U$551, U$639, U$727: (no value), buzzard_labels (22):PWR26
- added U$112, U$200, U$288, U$376, U$464, U$552, U$640, U$728: (no value), buzzard_labels (22):D1327
- added U$113, U$201, U$289, U$377, U$465, U$553, U$641, U$729: (no value), buzzard_labels (22):QWIIC31
- added U$114, U$202, U$290, U$378, U$466, U$554, U$642, U$730: (no value), buzzard_labels (22):A020
- added U$115, U$203, U$291, U$379, U$467, U$555, U$643, U$731: (no value), buzzard_labels (22):A121
- added U$116, U$204, U$292, U$380, U$468, U$556, U$644, U$732: (no value), buzzard_labels (22):A222
- added U$117, U$205, U$293, U$381, U$469, U$557, U$645, U$733: (no value), buzzard_labels (22):A323
- added U$118, U$206, U$294, U$382, U$470, U$558, U$646, U$734: (no value), buzzard_labels (22):A424
- added U$119, U$207, U$295, U$383, U$471, U$559, U$647, U$735: (no value), buzzard_labels (22):A525
- added U$120, U$208, U$296, U$384, U$472, U$560, U$648, U$736: (no value), buzzard_labels (22):VIN19
- added U$123, U$211, U$299, U$387, U$475, U$563, U$651, U$739: (no value), buzzard_labels (23):#RESET1
- added U$124, U$212, U$300, U$388, U$476, U$564, U$652, U$740: (no value), buzzard_labels (23):REF0
- added U$125, U$213, U$301, U$389, U$477, U$565, U$653, U$741: (no value), buzzard_labels (23):AREF2
- added U$126, U$214, U$302, U$390, U$478, U$566, U$654, U$742: (no value), buzzard_labels (23):GND7
- added U$127, U$215, U$303, U$391, U$479, U$567, U$655, U$743: (no value), buzzard_labels (23):MOSI4
- added U$128, U$216, U$304, U$392, U$480, U$568, U$656, U$744: (no value), buzzard_labels (23):3V36
- added U$129, U$217, U$305, U$393, U$481, U$569, U$657, U$745: (no value), buzzard_labels (23):SCK5
- added U$130, U$218, U$306, U$394, U$482, U$570, U$658, U$746: (no value), buzzard_labels (23):MISO3
- added U$131, U$219, U$307, U$395, U$483, U$571, U$659, U$747: (no value), buzzard_labels (24):RESET0
- added U$132, U$220, U$308, U$396, U$484, U$572, U$660, U$748: (no value), buzzard_labels (25):3V325
- added U$133, U$221, U$309, U$397, U$485, U$573, U$661, U$749: (no value), buzzard_labels (25):A018
- added U$134, U$222, U$310, U$398, U$486, U$574, U$662, U$750: (no value), buzzard_labels (25):A119
- added U$135, U$223, U$311, U$399, U$487, U$575, U$663, U$751: (no value), buzzard_labels (25):A220
- added U$136, U$224, U$312, U$400, U$488, U$576, U$664, U$752: (no value), buzzard_labels (25):A321
- added U$137, U$225, U$313, U$401, U$489, U$577, U$665, U$753: (no value), buzzard_labels (25):A422
- added U$138, U$226, U$314, U$402, U$490, U$578, U$666, U$754: (no value), buzzard_labels (25):A523
- added U$139, U$227, U$315, U$403, U$491, U$579, U$667, U$755: (no value), buzzard_labels (25):AREF2
- added U$140, U$228, U$316, U$404, U$492, U$580, U$668, U$756: (no value), buzzard_labels (25):D0#RX17
- added U$141, U$229, U$317, U$405, U$493, U$581, U$669, U$757: (no value), buzzard_labels (25):D1#TX15
- added U$142, U$230, U$318, U$406, U$494, U$582, U$670, U$758: (no value), buzzard_labels (25):D79
- added U$143, U$231, U$319, U$407, U$495, U$583, U$671, U$759: (no value), buzzard_labels (25):D88
- added U$144, U$232, U$320, U$408, U$496, U$584, U$672, U$760: (no value), buzzard_labels (25):D97
- added U$145, U$233, U$321, U$409, U$497, U$585, U$673, U$761: (no value), buzzard_labels (25):D106
- added U$146, U$234, U$322, U$410, U$498, U$586, U$674, U$762: (no value), buzzard_labels (25):D115
- added U$147, U$235, U$323, U$411, U$499, U$587, U$675, U$763: (no value), buzzard_labels (25):D124
- added U$148, U$236, U$324, U$412, U$500, U$588, U$676, U$764: (no value), buzzard_labels (25):D133
- added U$149, U$237, U$325, U$413, U$501, U$589, U$677, U$765: (no value), buzzard_labels (25):D214
- added U$150, U$238, U$326, U$414, U$502, U$590, U$678, U$766: (no value), buzzard_labels (25):D313
- added U$151, U$239, U$327, U$415, U$503, U$591, U$679, U$767: (no value), buzzard_labels (25):D412
- added U$152, U$240, U$328, U$416, U$504, U$592, U$680, U$768: (no value), buzzard_labels (25):D511
- added U$153, U$241, U$329, U$417, U$505, U$593, U$681, U$769: (no value), buzzard_labels (25):D610
- added U$154, U$155, U$156, U$242, U$243, U$244, U$330, U$331, U$332, U$418, U$419, U$420, U$506, U$507, U$508, U$594, U$595, U$596, U$682, U$683, U$684, U$770, U$771, U$772: (no value), buzzard_labels (25):GND24
- added U$157, U$245, U$333, U$421, U$509, U$597, U$685, U$773: (no value), buzzard_labels (25):GND33
- added U$158, U$246, U$334, U$422, U$510, U$598, U$686, U$774: (no value), buzzard_labels (25):MISO30
- added U$159, U$247, U$335, U$423, U$511, U$599, U$687, U$775: (no value), buzzard_labels (25):MOSI34
- added U$160, U$248, U$336, U$424, U$512, U$600, U$688, U$776: (no value), buzzard_labels (25):REF28
- added U$161, U$249, U$337, U$425, U$513, U$601, U$689, U$777: (no value), buzzard_labels (25):RESET32
- added U$162, U$250, U$338, U$426, U$514, U$602, U$690, U$778: (no value), buzzard_labels (25):SCK31
- added U$163, U$251, U$339, U$427, U$515, U$603, U$691, U$779: (no value), buzzard_labels (25):SCL0
- added U$164, U$252, U$340, U$428, U$516, U$604, U$692, U$780: (no value), buzzard_labels (25):SDA1
- added U$165, U$253, U$341, U$429, U$517, U$605, U$693, U$781: (no value), buzzard_labels (25):VIN27
- added U$166, U$254, U$342, U$430, U$518, U$606, U$694, U$782: (no value), buzzard_labels (26):#RESET1
- added U$167, U$255, U$343, U$431, U$519, U$607, U$695, U$783: (no value), buzzard_labels (26):3V30
- added U$168, U$256, U$344, U$432, U$520, U$608, U$696, U$784: (no value), buzzard_labels (25):5V26
- added U$169, U$257, U$345, U$433, U$521, U$609, U$697, U$785: (no value), buzzard_labels (27):RESET0
- added U$170, U$258, U$346, U$434, U$522, U$610, U$698, U$786: (no value), bitmap#jpg:BITMAP#JPG
- added U$171, U$259, U$347, U$435, U$523, U$611, U$699, U$787: (no value), buzzard_labels:440
- added U$172, U$260, U$348, U$436, U$524, U$612, U$700, U$788: (no value), buzzard_labels:REDBOARD_TURBO1
- added U$173, U$261, U$349, U$437, U$525, U$613, U$701, U$789: (no value), buzzard_labels (1):CHG_SET1
- added U$174, U$262, U$350, U$438, U$526, U$614, U$702, U$790: (no value), buzzard_labels:LED1
- added U$175, U$263, U$351, U$439, U$527, U$615, U$703, U$791: (no value), buzzard_labels:PWR0
- added U$176, U$264, U$352, U$440, U$528, U$616, U$704, U$792: (no value), buzzard_labels:VIN#_6V_MAX2
- added U$177, U$265, U$353, U$441, U$529, U$617, U$705, U$89: (no value), buzzard_labels (22):3V317
- added U$178, U$266, U$354, U$442, U$530, U$618, U$706, U$90: (no value), buzzard_labels (22):5V18
- added U$179, U$267, U$355, U$443, U$531, U$619, U$707, U$91: (no value), buzzard_labels (22):CHG30
- added U$180, U$268, U$356, U$444, U$532, U$620, U$708, U$92: (no value), buzzard_labels (22):RX#D015
- added U$181, U$269, U$357, U$445, U$533, U$621, U$709, U$93: (no value), buzzard_labels (22):TX#D114
- added U$182, U$270, U$358, U$446, U$534, U$622, U$710, U$94: (no value), buzzard_labels (22):D213
- added U$183, U$271, U$359, U$447, U$535, U$623, U$711, U$95: (no value), buzzard_labels (22):D312
- added U$184, U$272, U$360, U$448, U$536, U$624, U$712, U$96: (no value), buzzard_labels (22):D411
- added U$185, U$273, U$361, U$449, U$537, U$625, U$713, U$97: (no value), buzzard_labels (22):D510
- added U$186, U$274, U$362, U$450, U$538, U$626, U$714, U$98: (no value), buzzard_labels (22):D69
- added U$187, U$275, U$363, U$451, U$539, U$627, U$715, U$99: (no value), buzzard_labels (22):D78
- added U10, U15, U20, U25, U30, U35, U40, U45: W25Q32FV, SparkFun-IC-Memory:SOIC-8
- added U11, U16, U21, U26, U31, U36, U41, U6: ATSAMD21G-A, samd21-temp:TQFP-48
- added U12, U17, U22, U27, U32, U37, U42, U7: 3.3V, SparkFun-PowerIC:SOT23-5
- added U13, U18, U23, U28, U33, U38, U43, U8: 74AHC1G125, SparkFun-DigitalIC:SOT23-5
- added U14, U19, U24, U29, U34, U39, U44, U9: MCP73831, SparkFun-PowerIC:SOT23-5
- added Y2, Y3, Y4, Y5, Y6, Y7, Y8, Y9: 32.768kHz, samd21-temp:CRYSTAL-SMD-3.2X1.5MM
Connections:
- new net !RESET1: JP1.10, JP2.RESET@1, JP2.RESET@2, R13.1, S2.1, S2.2, U6.40
- new net !RESET2: JP5.10, JP8.RESET@1, JP8.RESET@2, R25.1, S3.1, S3.2, U11.40
- new net !RESET3: JP10.10, JP11.RESET@1, JP11.RESET@2, R37.1, S4.1, S4.2, U16.40
- new net !RESET4: JP13.10, JP14.RESET@1, JP14.RESET@2, R49.1, S5.1, S5.2, U21.40
- new net !RESET5: JP16.10, JP17.RESET@1, JP17.RESET@2, R61.1, S6.1, S6.2, U26.40
- new net !RESET6: JP19.10, JP20.RESET@1, JP20.RESET@2, R73.1, S7.1, S7.2, U31.40
- new net !RESET7: JP22.10, JP23.RESET@1, JP23.RESET@2, R85.1, S8.1, S8.2, U36.40
- new net !RESET8: JP25.10, JP26.RESET@1, JP26.RESET@2, R97.1, S9.1, S9.2, U41.40
- new net 3.3V1: C15.1, C18.1, C22.1, C23.1, C27.1, C28.1, D14.1, J5.2, JP1.1, JP2.3.3V, JP2.IOREF, JP2.VCC, L2.1, R13.2, R14.2, R15.2, R18.2, R20.2, U10.3, U10.7, U10.8, U6.17, U6.36, U6.44, U7.5
- new net 3.3V2: C29.1, C32.1, C36.1, C37.1, C41.1, C42.1, D21.1, J8.2, JP5.1, JP8.3.3V, JP8.IOREF, JP8.VCC, L3.1, R25.2, R26.2, R27.2, R30.2, R32.2, U11.17, U11.36, U11.44, U12.5, U15.3, U15.7, U15.8
- new net 3.3V3: C43.1, C46.1, C50.1, C51.1, C55.1, C56.1, D28.1, J11.2, JP10.1, JP11.3.3V, JP11.IOREF, JP11.VCC, L4.1, R37.2, R38.2, R39.2, R42.2, R44.2, U16.17, U16.36, U16.44, U17.5, U20.3, U20.7, U20.8
- new net 3.3V4: C57.1, C60.1, C64.1, C65.1, C69.1, C70.1, D35.1, J14.2, JP13.1, JP14.3.3V, JP14.IOREF, JP14.VCC, L5.1, R49.2, R50.2, R51.2, R54.2, R56.2, U21.17, U21.36, U21.44, U22.5, U25.3, U25.7, U25.8
- new net 3.3V5: C71.1, C74.1, C78.1, C79.1, C83.1, C84.1, D42.1, J17.2, JP16.1, JP17.3.3V, JP17.IOREF, JP17.VCC, L6.1, R61.2, R62.2, R63.2, R66.2, R68.2, U26.17, U26.36, U26.44, U27.5, U30.3, U30.7, U30.8
- new net 3.3V6: C85.1, C88.1, C92.1, C93.1, C97.1, C98.1, D49.1, J20.2, JP19.1, JP20.3.3V, JP20.IOREF, JP20.VCC, L7.1, R73.2, R74.2, R75.2, R78.2, R80.2, U31.17, U31.36, U31.44, U32.5, U35.3, U35.7, U35.8
- new net 3.3V7: C102.1, C106.1, C107.1, C111.1, C112.1, C99.1, D56.1, J23.2, JP22.1, JP23.3.3V, JP23.IOREF, JP23.VCC, L8.1, R85.2, R86.2, R87.2, R90.2, R92.2, U36.17, U36.36, U36.44, U37.5, U40.3, U40.7, U40.8
- new net 3.3V8: C113.1, C116.1, C120.1, C121.1, C125.1, C126.1, D63.1, J26.2, JP25.1, JP26.3.3V, JP26.IOREF, JP26.VCC, L9.1, R102.2, R104.2, R97.2, R98.2, R99.2, U41.17, U41.36, U41.44, U42.5, U45.3, U45.7, U45.8
- new net A10: JP2.A4, U6.10
- new net A11: JP2.A5, U6.47
- new net A12: JP8.A3, U11.9
- new net A13: JP8.A2, U11.8
- new net A14: JP8.A1, U11.7
- new net A15: JP8.A0, U11.3
- new net A16: JP8.A4, U11.10
- new net A17: JP8.A5, U11.47
- new net A18: JP11.A3, U16.9
- new net A19: JP11.A2, U16.8
- new net A20: JP11.A1, U16.7
- new net A21: JP11.A0, U16.3
- new net A22: JP11.A4, U16.10
- new net A23: JP11.A5, U16.47
- new net A24: JP14.A3, U21.9
- new net A25: JP14.A2, U21.8
- new net A26: JP14.A1, U21.7
- new net A27: JP14.A0, U21.3
- new net A28: JP14.A4, U21.10
- new net A29: JP14.A5, U21.47
- new net A30: JP17.A3, U26.9
- new net A31: JP17.A2, U26.8
- new net A32: JP17.A1, U26.7
- new net A33: JP17.A0, U26.3
- new net A34: JP17.A4, U26.10
- new net A35: JP17.A5, U26.47
- new net A36: JP20.A3, U31.9
- new net A37: JP20.A2, U31.8
- new net A38: JP20.A1, U31.7
- new net A39: JP20.A0, U31.3
- new net A40: JP20.A4, U31.10
- new net A41: JP20.A5, U31.47
- new net A42: JP23.A3, U36.9
- new net A43: JP23.A2, U36.8
- new net A44: JP23.A1, U36.7
- new net A45: JP23.A0, U36.3
- new net A46: JP23.A4, U36.10
- new net A47: JP23.A5, U36.47
- new net A48: JP26.A3, U41.9
- new net A49: JP26.A2, U41.8
- new net A50: JP26.A1, U41.7
- new net A51: JP26.A0, U41.3
- new net A52: JP26.A4, U41.10
- new net A53: JP26.A5, U41.47
- new net A6: JP2.A3, U6.9
- new net A7: JP2.A2, U6.8
- new net A8: JP2.A1, U6.7
- new net A9: JP2.A0, U6.3
- new net AREF1: JP2.AREF, U6.4
- new net AREF2: JP8.AREF, U11.4
- new net AREF3: JP11.AREF, U16.4
- new net AREF4: JP14.AREF, U21.4
- new net AREF5: JP17.AREF, U26.4
- new net AREF6: JP20.AREF, U31.4
- new net AREF7: JP23.AREF, U36.4
- new net AREF8: JP26.AREF, U41.4
- new net CHG_STAT1: R22.2, U9.1
- new net CHG_STAT2: R34.2, U14.1
- new net CHG_STAT3: R46.2, U19.1
- new net CHG_STAT4: R58.2, U24.1
- new net CHG_STAT5: R70.2, U29.1
- new net CHG_STAT6: R82.2, U34.1
- new net CHG_STAT7: R94.2, U39.1
- new net CHG_STAT8: R106.2, U44.1
- new net D0/RXI1: JP2.D0, U6.16
- new net D0/RXI2: JP8.D0, U11.16
- new net D0/RXI3: JP11.D0, U16.16
- new net D0/RXI4: JP14.D0, U21.16
- new net D0/RXI5: JP17.D0, U26.16
- new net D0/RXI6: JP20.D0, U31.16
- new net D0/RXI7: JP23.D0, U36.16
- new net D0/RXI8: JP26.D0, U41.16
- new net D1: JP2.D4, U6.13
- new net D1/TXO1: JP2.D1, U6.15
- new net D1/TXO2: JP8.D1, U11.15
- new net D1/TXO3: JP11.D1, U16.15
- new net D1/TXO4: JP14.D1, U21.15
- new net D1/TXO5: JP17.D1, U26.15
- new net D1/TXO6: JP20.D1, U31.15
- new net D1/TXO7: JP23.D1, U36.15
- new net D1/TXO8: JP26.D1, U41.15
- new net D100: JP26.D5, U41.24
- new net D101: JP26.D6, U41.29
- new net D102: JP26.D7, U41.30
- new net D103: JP26.D8, U41.11
- new net D104: JP26.D9, U41.12
- new net D105: JP26.D12, U41.28
- new net D106: JP26.D11, U41.25
- new net D107: JP26.D10, U41.27
- new net D108: JP26.D13, Q17.1, R108.2, U41.26
- new net D14: JP2.D3, U6.14
- new net D15: JP2.D2, U6.23
- new net D16: JP2.D5, U6.24
- new net D17: JP2.D6, U6.29
- new net D18: JP2.D7, U6.30
- new net D19: JP2.D8, U6.11
- new net D20: JP2.D9, U6.12
- new net D21: JP2.D12, U6.28
- new net D22: JP2.D11, U6.25
- new net D23: JP2.D10, U6.27
- new net D24: JP2.D13, Q3.1, R24.2, U6.26
- new net D25: JP8.D4, U11.13
- new net D26: JP8.D3, U11.14
- new net D27: JP8.D2, U11.23
- new net D28: JP8.D5, U11.24
- new net D29: JP8.D6, U11.29
- new net D30: JP8.D7, U11.30
- new net D31: JP8.D8, U11.11
- new net D32: JP8.D9, U11.12
- new net D33: JP8.D12, U11.28
- new net D34: JP8.D11, U11.25
- new net D35: JP8.D10, U11.27
- new net D36: JP8.D13, Q5.1, R36.2, U11.26
- new net D37: JP11.D4, U16.13
- new net D38: JP11.D3, U16.14
- new net D39: JP11.D2, U16.23
- new net D40: JP11.D5, U16.24
- new net D41: JP11.D6, U16.29
- new net D42: JP11.D7, U16.30
- new net D43: JP11.D8, U16.11
- new net D44: JP11.D9, U16.12
- new net D45: JP11.D12, U16.28
- new net D46: JP11.D11, U16.25
- new net D47: JP11.D10, U16.27
- new net D48: JP11.D13, Q7.1, R48.2, U16.26
- new net D49: JP14.D4, U21.13
- new net D50: JP14.D3, U21.14
- new net D51: JP14.D2, U21.23
- new net D52: JP14.D5, U21.24
- new net D53: JP14.D6, U21.29
- new net D54: JP14.D7, U21.30
- new net D55: JP14.D8, U21.11
- new net D56: JP14.D9, U21.12
- new net D57: JP14.D12, U21.28
- new net D58: JP14.D11, U21.25
- new net D59: JP14.D10, U21.27
- new net D60: JP14.D13, Q9.1, R60.2, U21.26
- new net D61: JP17.D4, U26.13
- new net D62: JP17.D3, U26.14
- new net D63: JP17.D2, U26.23
- new net D64: JP17.D5, U26.24
- new net D65: JP17.D6, U26.29
- new net D66: JP17.D7, U26.30
- new net D67: JP17.D8, U26.11
- new net D68: JP17.D9, U26.12
- new net D69: JP17.D12, U26.28
- new net D70: JP17.D11, U26.25
- new net D71: JP17.D10, U26.27
- new net D72: JP17.D13, Q11.1, R72.2, U26.26
- new net D73: JP20.D4, U31.13
- new net D74: JP20.D3, U31.14
- new net D75: JP20.D2, U31.23
- new net D76: JP20.D5, U31.24
- new net D77: JP20.D6, U31.29
- new net D78: JP20.D7, U31.30
- new net D79: JP20.D8, U31.11
- new net D80: JP20.D9, U31.12
- new net D81: JP20.D12, U31.28
- new net D82: JP20.D11, U31.25
- new net D83: JP20.D10, U31.27
- new net D84: JP20.D13, Q13.1, R84.2, U31.26
- new net D85: JP23.D4, U36.13
- new net D86: JP23.D3, U36.14
- new net D87: JP23.D2, U36.23
- new net D88: JP23.D5, U36.24
- new net D89: JP23.D6, U36.29
- new net D90: JP23.D7, U36.30
- new net D91: JP23.D8, U36.11
- new net D92: JP23.D9, U36.12
- new net D93: JP23.D12, U36.28
- new net D94: JP23.D11, U36.25
- new net D95: JP23.D10, U36.27
- new net D96: JP23.D13, Q15.1, R96.2, U36.26
- new net D97: JP26.D4, U41.13
- new net D98: JP26.D3, U41.14
- new net D99: JP26.D2, U41.23
- new net FLASH_CS1: U10.1, U6.22
- new net FLASH_CS2: U11.22, U15.1
- new net FLASH_CS3: U16.22, U20.1
- new net FLASH_CS4: U21.22, U25.1
- new net FLASH_CS5: U26.22, U30.1
- new net FLASH_CS6: U31.22, U35.1
- new net FLASH_CS7: U36.22, U40.1
- new net FLASH_CS8: U41.22, U45.1
- new net FLASH_MISO1: U10.2, U6.48
- new net FLASH_MISO2: U11.48, U15.2
- new net FLASH_MISO3: U16.48, U20.2
- new net FLASH_MISO4: U21.48, U25.2
- new net FLASH_MISO5: U26.48, U30.2
- new net FLASH_MISO6: U31.48, U35.2
- new net FLASH_MISO7: U36.48, U40.2
- new net FLASH_MISO8: U41.48, U45.2
- new net FLASH_MOSI1: U10.5, U6.37
- new net FLASH_MOSI2: U11.37, U15.5
- new net FLASH_MOSI3: U16.37, U20.5
- new net FLASH_MOSI4: U21.37, U25.5
- new net FLASH_MOSI5: U26.37, U30.5
- new net FLASH_MOSI6: U31.37, U35.5
- new net FLASH_MOSI7: U36.37, U40.5
- new net FLASH_MOSI8: U41.37, U45.5
- new net FLASH_SCK1: U10.6, U6.38
- new net FLASH_SCK2: U11.38, U15.6
- new net FLASH_SCK3: U16.38, U20.6
- new net FLASH_SCK4: U21.38, U25.6
- new net FLASH_SCK5: U26.38, U30.6
- new net FLASH_SCK6: U31.38, U35.6
- new net FLASH_SCK7: U36.38, U40.6
- new net FLASH_SCK8: U41.38, U45.6
- new net GND1: C15.2, C16.2, C17.2, C18.2, C19.1, C20.2, C21.2, C22.2, C23.2, C24.2, C25.2, C26.2, C27.2, C28.2, D14.3, J4.1, J5.1, J6.GND, J6.SHIELD, J6.SHIELD10, J6.SHIELD2, J6.SHIELD3, J6.SHIELD4, J6.SHIELD5, J6.SHIELD6, J6.SHIELD7, J6.SHIELD8, J6.SHIELD9, JP1.3, JP1.5, JP2.GND@1, JP2.GND@2, JP2.GND@3, JP2.GND@4, JP4.GND, JP4.GNDBREAK, Q3.2, R21.1, R23.1, R24.1, S2.3, S2.4, SJ2.1, U10.4, U6.18, U6.35, U6.42, U6.5, U7.2, U8.3, U9.2
- new net GND2: C29.2, C30.2, C31.2, C32.2, C33.1, C34.2, C35.2, C36.2, C37.2, C38.2, C39.2, C40.2, C41.2, C42.2, D21.3, J7.1, J8.1, J9.GND, J9.SHIELD, J9.SHIELD10, J9.SHIELD2, J9.SHIELD3, J9.SHIELD4, J9.SHIELD5, J9.SHIELD6, J9.SHIELD7, J9.SHIELD8, J9.SHIELD9, JP5.3, JP5.5, JP8.GND@1, JP8.GND@2, JP8.GND@3, JP8.GND@4, JP9.GND, JP9.GNDBREAK, Q5.2, R33.1, R35.1, R36.1, S3.3, S3.4, SJ3.1, U11.18, U11.35, U11.42, U11.5, U12.2, U13.3, U14.2, U15.4
- new net GND3: C43.2, C44.2, C45.2, C46.2, C47.1, C48.2, C49.2, C50.2, C51.2, C52.2, C53.2, C54.2, C55.2, C56.2, D28.3, J10.1, J11.1, J12.GND, J12.SHIELD, J12.SHIELD10, J12.SHIELD2, J12.SHIELD3, J12.SHIELD4, J12.SHIELD5, J12.SHIELD6, J12.SHIELD7, J12.SHIELD8, J12.SHIELD9, JP10.3, JP10.5, JP11.GND@1, JP11.GND@2, JP11.GND@3, JP11.GND@4, JP12.GND, JP12.GNDBREAK, Q7.2, R45.1, R47.1, R48.1, S4.3, S4.4, SJ4.1, U16.18, U16.35, U16.42, U16.5, U17.2, U18.3, U19.2, U20.4
- new net GND4: C57.2, C58.2, C59.2, C60.2, C61.1, C62.2, C63.2, C64.2, C65.2, C66.2, C67.2, C68.2, C69.2, C70.2, D35.3, J13.1, J14.1, J15.GND, J15.SHIELD, J15.SHIELD10, J15.SHIELD2, J15.SHIELD3, J15.SHIELD4, J15.SHIELD5, J15.SHIELD6, J15.SHIELD7, J15.SHIELD8, J15.SHIELD9, JP13.3, JP13.5, JP14.GND@1, JP14.GND@2, JP14.GND@3, JP14.GND@4, JP15.GND, JP15.GNDBREAK, Q9.2, R57.1, R59.1, R60.1, S5.3, S5.4, SJ5.1, U21.18, U21.35, U21.42, U21.5, U22.2, U23.3, U24.2, U25.4
- new net GND5: C71.2, C72.2, C73.2, C74.2, C75.1, C76.2, C77.2, C78.2, C79.2, C80.2, C81.2, C82.2, C83.2, C84.2, D42.3, J16.1, J17.1, J18.GND, J18.SHIELD, J18.SHIELD10, J18.SHIELD2, J18.SHIELD3, J18.SHIELD4, J18.SHIELD5, J18.SHIELD6, J18.SHIELD7, J18.SHIELD8, J18.SHIELD9, JP16.3, JP16.5, JP17.GND@1, JP17.GND@2, JP17.GND@3, JP17.GND@4, JP18.GND, JP18.GNDBREAK, Q11.2, R69.1, R71.1, R72.1, S6.3, S6.4, SJ6.1, U26.18, U26.35, U26.42, U26.5, U27.2, U28.3, U29.2, U30.4
- new net GND6: C85.2, C86.2, C87.2, C88.2, C89.1, C90.2, C91.2, C92.2, C93.2, C94.2, C95.2, C96.2, C97.2, C98.2, D49.3, J19.1, J20.1, J21.GND, J21.SHIELD, J21.SHIELD10, J21.SHIELD2, J21.SHIELD3, J21.SHIELD4, J21.SHIELD5, J21.SHIELD6, J21.SHIELD7, J21.SHIELD8, J21.SHIELD9, JP19.3, JP19.5, JP20.GND@1, JP20.GND@2, JP20.GND@3, JP20.GND@4, JP21.GND, JP21.GNDBREAK, Q13.2, R81.1, R83.1, R84.1, S7.3, S7.4, SJ7.1, U31.18, U31.35, U31.42, U31.5, U32.2, U33.3, U34.2, U35.4
- new net GND7: C100.2, C101.2, C102.2, C103.1, C104.2, C105.2, C106.2, C107.2, C108.2, C109.2, C110.2, C111.2, C112.2, C99.2, D56.3, J22.1, J23.1, J24.GND, J24.SHIELD, J24.SHIELD10, J24.SHIELD2, J24.SHIELD3, J24.SHIELD4, J24.SHIELD5, J24.SHIELD6, J24.SHIELD7, J24.SHIELD8, J24.SHIELD9, JP22.3, JP22.5, JP23.GND@1, JP23.GND@2, JP23.GND@3, JP23.GND@4, JP24.GND, JP24.GNDBREAK, Q15.2, R93.1, R95.1, R96.1, S8.3, S8.4, SJ8.1, U36.18, U36.35, U36.42, U36.5, U37.2, U38.3, U39.2, U40.4
- new net GND8: C113.2, C114.2, C115.2, C116.2, C117.1, C118.2, C119.2, C120.2, C121.2, C122.2, C123.2, C124.2, C125.2, C126.2, D63.3, J25.1, J26.1, J27.GND, J27.SHIELD, J27.SHIELD10, J27.SHIELD2, J27.SHIELD3, J27.SHIELD4, J27.SHIELD5, J27.SHIELD6, J27.SHIELD7, J27.SHIELD8, J27.SHIELD9, JP25.3, JP25.5, JP26.GND@1, JP26.GND@2, JP26.GND@3, JP26.GND@4, JP27.GND, JP27.GNDBREAK, Q17.2, R105.1, R107.1, R108.1, S9.3, S9.4, SJ9.1, U41.18, U41.35, U41.42, U41.5, U42.2, U43.3, U44.2, U45.4
- new net LED/SWCLK1: D14.4, JP1.4, U6.45
- new net LED/SWCLK2: D21.4, JP5.4, U11.45
- new net LED/SWCLK3: D28.4, JP10.4, U16.45
- new net LED/SWCLK4: D35.4, JP13.4, U21.45
- new net LED/SWCLK5: D42.4, JP16.4, U26.45
- new net LED/SWCLK6: D49.4, JP19.4, U31.45
- new net LED/SWCLK7: D56.4, JP22.4, U36.45
- new net LED/SWCLK8: D63.4, JP25.4, U41.45
- new net N$14: D9.A, R14.1
- new net N$15: D10.A, R15.1
- new net N$16: D10.C, Q3.3
- new net N$17: F2.1, J6.VBUS
- new net N$18: D8.A, R18.1
- new net N$19: D11.A, R20.1
- new net N$20: D9.C, SJ2.2
- new net N$21: R21.2, R23.2, U9.5
- new net N$22: D12.C, R22.1
- new net N$23: C33.2, U11.1, Y3.P$2
- new net N$24: C34.1, U11.2, Y3.P$1
- new net N$25: D16.A, R26.1
- new net N$26: D17.A, R27.1
- new net N$27: D17.C, Q5.3
- new net N$28: F3.1, J9.VBUS
- new net N$29: D15.A, R30.1
- new net N$30: D18.A, R32.1
- new net N$31: D16.C, SJ3.2
- new net N$32: R33.2, R35.2, U14.5
- new net N$33: D19.C, R34.1
- new net N$34: C47.2, U16.1, Y4.P$2
- new net N$35: C48.1, U16.2, Y4.P$1
- new net N$36: D23.A, R38.1
- new net N$37: D24.A, R39.1
- new net N$38: D24.C, Q7.3
- new net N$39: F4.1, J12.VBUS
- new net N$40: D22.A, R42.1
- new net N$41: D25.A, R44.1
- new net N$42: D23.C, SJ4.2
- new net N$43: R45.2, R47.2, U19.5
- new net N$44: D26.C, R46.1
- new net N$45: C61.2, U21.1, Y5.P$2
- new net N$46: C62.1, U21.2, Y5.P$1
- new net N$47: D30.A, R50.1
- new net N$48: D31.A, R51.1
- new net N$49: D31.C, Q9.3
- new net N$50: F5.1, J15.VBUS
- new net N$51: D29.A, R54.1
- new net N$52: D32.A, R56.1
- new net N$53: D30.C, SJ5.2
- new net N$54: R57.2, R59.2, U24.5
- new net N$55: D33.C, R58.1
- new net N$56: C75.2, U26.1, Y6.P$2
- new net N$57: C76.1, U26.2, Y6.P$1
- new net N$58: D37.A, R62.1
- new net N$59: D38.A, R63.1
- new net N$60: D38.C, Q11.3
- new net N$61: F6.1, J18.VBUS
- new net N$62: D36.A, R66.1
- new net N$63: D39.A, R68.1
- new net N$64: D37.C, SJ6.2
- new net N$65: R69.2, R71.2, U29.5
- new net N$66: D40.C, R70.1
- new net N$67: C89.2, U31.1, Y7.P$2
- new net N$68: C90.1, U31.2, Y7.P$1
- new net N$69: D44.A, R74.1
- new net N$7: C19.2, U6.1, Y2.P$2
- new net N$70: D45.A, R75.1
- new net N$71: D45.C, Q13.3
- new net N$72: F7.1, J21.VBUS
- new net N$73: D43.A, R78.1
- new net N$74: D46.A, R80.1
- new net N$75: D44.C, SJ7.2
- new net N$76: R81.2, R83.2, U34.5
- new net N$77: D47.C, R82.1
- new net N$78: C103.2, U36.1, Y8.P$2
- new net N$79: C104.1, U36.2, Y8.P$1
- new net N$80: D51.A, R86.1
- new net N$81: D52.A, R87.1
- new net N$82: D52.C, Q15.3
- new net N$83: F8.1, J24.VBUS
- new net N$84: D50.A, R90.1
- new net N$85: D53.A, R92.1
- new net N$86: D51.C, SJ8.2
- new net N$87: R93.2, R95.2, U39.5
- new net N$88: D54.C, R94.1
- new net N$89: C117.2, U41.1, Y9.P$2
- new net N$9: C20.1, U6.2, Y2.P$1
- new net N$90: C118.1, U41.2, Y9.P$1
- new net N$91: D58.A, R98.1
- new net N$92: D59.A, R99.1
- new net N$93: D59.C, Q17.3
- new net N$94: F9.1, J27.VBUS
- new net N$95: D57.A, R102.1
- new net N$96: D60.A, R104.1
- new net N$97: D58.C, SJ9.2
- new net N$98: R105.2, R107.2, U44.5
- new net N$99: D61.C, R106.1
- new net RX_LED/SWDIO1: D11.C, JP1.2, TP2.P$1, U6.46
- new net RX_LED/SWDIO2: D18.C, JP5.2, TP3.P$1, U11.46
- new net RX_LED/SWDIO3: D25.C, JP10.2, TP4.P$1, U16.46
- new net RX_LED/SWDIO4: D32.C, JP13.2, TP5.P$1, U21.46
- new net RX_LED/SWDIO5: D39.C, JP16.2, TP6.P$1, U26.46
- new net RX_LED/SWDIO6: D46.C, JP19.2, TP7.P$1, U31.46
- new net RX_LED/SWDIO7: D53.C, JP22.2, TP8.P$1, U36.46
- new net RX_LED/SWDIO8: D60.C, JP25.2, TP9.P$1, U41.46
- new net SCL1: J5.4, JP2.SCL, U6.32
- new net SCL2: J8.4, JP8.SCL, U11.32
- new net SCL3: J11.4, JP11.SCL, U16.32
- new net SCL4: J14.4, JP14.SCL, U21.32
- new net SCL5: J17.4, JP17.SCL, U26.32
- new net SCL6: J20.4, JP20.SCL, U31.32
- new net SCL7: J23.4, JP23.SCL, U36.32
- new net SCL8: J26.4, JP26.SCL, U41.32
- new net SDA1: J5.3, JP2.SDA, U6.31
- new net SDA2: J8.3, JP8.SDA, U11.31
- new net SDA3: J11.3, JP11.SDA, U16.31
- new net SDA4: J14.3, JP14.SDA, U21.31
- new net SDA5: J17.3, JP17.SDA, U26.31
- new net SDA6: J20.3, JP20.SDA, U31.31
- new net SDA7: J23.3, JP23.SDA, U36.31
- new net SDA8: J26.3, JP26.SDA, U41.31
- new net SPI_MISO1: JP2.MISO, U6.21
- new net SPI_MISO2: JP8.MISO, U11.21
- new net SPI_MISO3: JP11.MISO, U16.21
- new net SPI_MISO4: JP14.MISO, U21.21
- new net SPI_MISO5: JP17.MISO, U26.21
- new net SPI_MISO6: JP20.MISO, U31.21
- new net SPI_MISO7: JP23.MISO, U36.21
- new net SPI_MISO8: JP26.MISO, U41.21
- new net SPI_MOSI1: JP2.MOSI, U6.19
- new net SPI_MOSI2: JP8.MOSI, U11.19
- new net SPI_MOSI3: JP11.MOSI, U16.19
- new net SPI_MOSI4: JP14.MOSI, U21.19
- new net SPI_MOSI5: JP17.MOSI, U26.19
- new net SPI_MOSI6: JP20.MOSI, U31.19
- new net SPI_MOSI7: JP23.MOSI, U36.19
- new net SPI_MOSI8: JP26.MOSI, U41.19
- new net SPI_SCK1: JP2.SCK, U6.20
- new net SPI_SCK2: JP8.SCK, U11.20
- new net SPI_SCK3: JP11.SCK, U16.20
- new net SPI_SCK4: JP14.SCK, U21.20
- new net SPI_SCK5: JP17.SCK, U26.20
- new net SPI_SCK6: JP20.SCK, U31.20
- new net SPI_SCK7: JP23.SCK, U36.20
- new net SPI_SCK8: JP26.SCK, U41.20
- new net TX_LED1: D8.C, U6.39
- new net TX_LED2: D15.C, U11.39
- new net TX_LED3: D22.C, U16.39
- new net TX_LED4: D29.C, U21.39
- new net TX_LED5: D36.C, U26.39
- new net TX_LED6: D43.C, U31.39
- new net TX_LED7: D50.C, U36.39
- new net TX_LED8: D57.C, U41.39
- new net USB_D+1: J6.D+, U6.34
- new net USB_D+2: J9.D+, U11.34
- new net USB_D+3: J12.D+, U16.34
- new net USB_D+4: J15.D+, U21.34
- new net USB_D+5: J18.D+, U26.34
- new net USB_D+6: J21.D+, U31.34
- new net USB_D+7: J24.D+, U36.34
- new net USB_D+8: J27.D+, U41.34
- new net USB_D-1: J6.D-, U6.33
- new net USB_D-2: J9.D-, U11.33
- new net USB_D-3: J12.D-, U16.33
- new net USB_D-4: J15.D-, U21.33
- new net USB_D-5: J18.D-, U26.33
- new net USB_D-6: J21.D-, U31.33
- new net USB_D-7: J24.D-, U36.33
- new net USB_D-8: J27.D-, U41.33
- new net USB_HOST_EN1: R17.1, U6.41
- new net USB_HOST_EN2: R29.1, U11.41
- new net USB_HOST_EN3: R41.1, U16.41
- new net USB_HOST_EN4: R53.1, U21.41
- new net USB_HOST_EN5: R65.1, U26.41
- new net USB_HOST_EN6: R77.1, U31.41
- new net USB_HOST_EN7: R89.1, U36.41
- new net USB_HOST_EN8: R101.1, U41.41
- new net USB_HOST_POWER_EN1: Q4.1, R19.1, U8.4
- new net USB_HOST_POWER_EN2: Q6.1, R31.1, U13.4
- new net USB_HOST_POWER_EN3: Q8.1, R43.1, U18.4
- new net USB_HOST_POWER_EN4: Q10.1, R55.1, U23.4
- new net USB_HOST_POWER_EN5: Q12.1, R67.1, U28.4
- new net USB_HOST_POWER_EN6: Q14.1, R79.1, U33.4
- new net USB_HOST_POWER_EN7: Q16.1, R91.1, U38.4
- new net USB_HOST_POWER_EN8: Q18.1, R103.1, U43.4
- new net USB_ID1: J6.ID, R16.1, R17.2, U8.1, U8.2
- new net USB_ID2: J9.ID, R28.1, R29.2, U13.1, U13.2
- new net USB_ID3: J12.ID, R40.1, R41.2, U18.1, U18.2
- new net USB_ID4: J15.ID, R52.1, R53.2, U23.1, U23.2
- new net USB_ID5: J18.ID, R64.1, R65.2, U28.1, U28.2
- new net USB_ID6: J21.ID, R76.1, R77.2, U33.1, U33.2
- new net USB_ID7: J24.ID, R88.1, R89.2, U38.1, U38.2
- new net USB_ID8: J27.ID, R100.1, R101.2, U43.1, U43.2
- new net VBAT1: C25.1, D13.A, J4.2, U9.3
- new net VBAT2: C39.1, D20.A, J7.2, U14.3
- new net VBAT3: C53.1, D27.A, J10.2, U19.3
- new net VBAT4: C67.1, D34.A, J13.2, U24.3
- new net VBAT5: C81.1, D41.A, J16.2, U29.3
- new net VBAT6: C95.1, D48.A, J19.2, U34.3
- new net VBAT7: C109.1, D55.A, J22.2, U39.3
- new net VBAT8: C123.1, D62.A, J25.2, U44.3
- new net VDDANA1: C17.1, L2.2, U6.6
- new net VDDANA2: C31.1, L3.2, U11.6
- new net VDDANA3: C45.1, L4.2, U16.6
- new net VDDANA4: C59.1, L5.2, U21.6
- new net VDDANA5: C73.1, L6.2, U26.6
- new net VDDANA6: C87.1, L7.2, U31.6
- new net VDDANA7: C101.1, L8.2, U36.6
- new net VDDANA8: C115.1, L9.2, U41.6
- new net VDDCORE1: C16.1, U6.43
- new net VDDCORE2: C30.1, U11.43
- new net VDDCORE3: C44.1, U16.43
- new net VDDCORE4: C58.1, U21.43
- new net VDDCORE5: C72.1, U26.43
- new net VDDCORE6: C86.1, U31.43
- new net VDDCORE7: C100.1, U36.43
- new net VDDCORE8: C114.1, U41.43
- new net VIN1: C21.1, C26.1, D12.A, D13.C, JP2.VIN, JP4.PWR, Q4.2, R16.2, R19.2, U7.1, U7.3, U8.5, U9.4
- new net VIN2: C35.1, C40.1, D19.A, D20.C, JP8.VIN, JP9.PWR, Q6.2, R28.2, R31.2, U12.1, U12.3, U13.5, U14.4
- new net VIN3: C49.1, C54.1, D26.A, D27.C, JP11.VIN, JP12.PWR, Q8.2, R40.2, R43.2, U17.1, U17.3, U18.5, U19.4
- new net VIN4: C63.1, C68.1, D33.A, D34.C, JP14.VIN, JP15.PWR, Q10.2, R52.2, R55.2, U22.1, U22.3, U23.5, U24.4
- new net VIN5: C77.1, C82.1, D40.A, D41.C, JP17.VIN, JP18.PWR, Q12.2, R64.2, R67.2, U27.1, U27.3, U28.5, U29.4
- new net VIN6: C91.1, C96.1, D47.A, D48.C, JP20.VIN, JP21.PWR, Q14.2, R76.2, R79.2, U32.1, U32.3, U33.5, U34.4
- new net VIN7: C105.1, C110.1, D54.A, D55.C, JP23.VIN, JP24.PWR, Q16.2, R88.2, R91.2, U37.1, U37.3, U38.5, U39.4
- new net VIN8: C119.1, C124.1, D61.A, D62.C, JP26.VIN, JP27.PWR, Q18.2, R100.2, R103.2, U42.1, U42.3, U43.5, U44.4
- new net VUSB1: C24.1, F2.2, JP2.5V, Q4.3
- new net VUSB2: C38.1, F3.2, JP8.5V, Q6.3
- new net VUSB3: C52.1, F4.2, JP11.5V, Q8.3
- new net VUSB4: C66.1, F5.2, JP14.5V, Q10.3
- new net VUSB5: C80.1, F6.2, JP17.5V, Q12.3
- new net VUSB6: C94.1, F7.2, JP20.5V, Q14.3
- new net VUSB7: C108.1, F8.2, JP23.5V, Q16.3
- new net VUSB8: C122.1, F9.2, JP26.5V, Q18.3
Routing:
- net 3.3V3: track 0.00 -> 230.3 mm, vias 0 -> 12
- net 3.3V4: track 0.00 -> 230.3 mm, vias 0 -> 12
- net 3.3V6: track 0.00 -> 230.3 mm, vias 0 -> 12
- net 3.3V5: track 0.00 -> 230.3 mm, vias 0 -> 12
- net 3.3V2: track 0.00 -> 230.3 mm, vias 0 -> 12
- net 3.3V1: track 0.00 -> 230.3 mm, vias 0 -> 12
- net 3.3V8: track 0.00 -> 230.3 mm, vias 0 -> 12
- net 3.3V7: track 0.00 -> 230.3 mm, vias 0 -> 12
- net VIN8: track 0.00 -> 127.8 mm, vias 0 -> 5
- net VIN5: track 0.00 -> 127.8 mm, vias 0 -> 5
- net VIN7: track 0.00 -> 127.8 mm, vias 0 -> 5
- net VIN4: track 0.00 -> 127.8 mm, vias 0 -> 5
- net VIN2: track 0.00 -> 127.8 mm, vias 0 -> 5
- net VIN1: track 0.00 -> 127.8 mm, vias 0 -> 5
- net VIN3: track 0.00 -> 127.8 mm, vias 0 -> 5
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- added copper zone on layer 1, net GND1
- added copper zone on layer 16, net GND1
- added copper zone on layer 1, net GND2
- added copper zone on layer 16, net GND2
- added copper zone on layer 1, net GND3
- added copper zone on layer 16, net GND3
- added copper zone on layer 1, net GND4
- added copper zone on layer 16, net GND4
- added copper zone on layer 1, net GND5
- added copper zone on layer 16, net GND5
- added copper zone on layer 1, net GND6
- added copper zone on layer 16, net GND6
- added copper zone on layer 1, net GND7
- added copper zone on layer 16, net GND7
- added copper zone on layer 1, net GND8
- added copper zone on layer 16, net GND8
Other:
- board size 58.4 x 53.3 mm -> 209.5 x 174.8 mm
- board text added: "Route Out"
- board text added: "v-score"
- board text removed: "Jim Lindblom"
- board text removed: "Revised by Mike Hord"
- board text removed: "Units in inches"
